File: esp32-c3-bare-bones-mini.kicad_sch (KiCad schematic)
At the start: 18 parts, among them J3 BATT, U1 ESP32-C3-MINI-1

Commit message: Dual-Mode Power
Parts:
- removed D1: ~, easyeda2kicad:SOD-323_L1.7-W1.3-LS2.6-RD, symbol easyeda2kicad:BZT52C3V6S_C19077438
- removed F1: ~, easyeda2kicad:F0805, symbol easyeda2kicad:SMD0805-050
- added C6, C7: 1uF 16V 10%, easyeda2kicad:C0805, symbol easyeda2kicad:CL21B105KOFNNNE
- added C8, C9: 47uf 10V 20%, CL31A476MPHNNNE:C1206, symbol CL31A476MPHNNNE:CL31A476MPHNNNE
- added SW3: Slide Switch, G-Switch MS-22D28-G020:SW-SMD_MS-22D28-G020, symbol G-Switch MS-22D28-G020:MS-22D28-G020
- added U2: LDO, RT9080-33GJ5:TSOT-23-5_RIT-M, symbol RT9080-33GJ5:RT9080-33GJ5
Connections:
- net GND: now also C6.1, C7.2, C8.2, C9.2, SW3.6, U2.2 (GND)
- net VCC_3V3: now also J1.2 (Pin_2), C8.1, C9.1, SW3.2
- net FUSE_VCC renamed VCC_IN
- net VCC_IN: now also C6.2, SW3.3, SW3.4, U2.1 (VIN); no longer J1.2 (Pin_2)
- new net: C7.1, SW3.1, U2.5 (VOUT)
- new net LDO_EN: SW3.5, U2.3 (EN)
Other:
- note added: "Power"
- note removed: "Over Voltage Protection"
